File: PCB/Schematico.brd (EAGLE design)
At the start: 91.5 x 98 mm, 26 parts, among them IC3 AT24CP

Commit message: OLED Measurement interface finished
Parts:
- moved JP5 28.7 mm to (57.3, 53.2)
- moved D1 11.5 mm to (42.3, 67.8), turned to 270 degrees
- moved IC2 5.10 mm to (52.5, 73.5)
- moved S3 5.00 mm to (52.3, 84.8)
- moved IC1 4.81 mm to (56.4, 69.2)
- moved JP9 4.57 mm to (77.5, 59.9)
- moved C3 4.47 mm to (64.3, 77.0)
- moved C4 4.26 mm to (66.8, 65.3)
- moved J1 4.12 mm to (62.8, 87.7)
- moved C1 2.83 mm to (44.3, 79.0)
- moved C5 2.06 mm to (47.4, 64.0)
Routing:
- net 5V: track 189.4 -> 207.6 mm
- net TX3V3: track 29.8 -> 34.7 mm
- net RX3V3: track 30.0 -> 34.7 mm
- net SDA3V3: track 24.3 -> 28.8 mm
- net BTLVL: track 89.6 -> 85.1 mm
- net SCL3V3: track 28.7 -> 32.9 mm
- net 3V3: track 47.2 -> 50.7 mm
- net VBAT: track 29.4 -> 26.7 mm
- net N$1: track 11.8 -> 13.8 mm
Other:
- board size 91.5 x 98 mm -> 91.5 x 100 mm
